File: Beta 1.0.97/eagle/tracker03-09.brd (EAGLE design)
At the start: 64.4 x 49.5 mm, 29 parts, among them IC1 7805, J1 ARRDUINO I, J2 7V-12V

Commit message: major update
Parts:
- added JP10, JP11, JP12, JP9: (no value), pinhead:1X02
- moved IC1 21.1 mm to (6.99, 48.9), turned to 0 degrees
- moved C2 17.1 mm to (5.71, 36.2)
- moved C3 15.1 mm to (18.4, 45.7), turned to 270 degrees
- moved C1 14.6 mm to (7.62, 42.5), turned to 0 degrees
- moved C4 12.6 mm to (14.0, 44.5), turned to 270 degrees
- moved R3 3.81 mm to (34.3, 12.7)
- moved R4 3.81 mm to (29.2, 12.7)
- moved SJ1 3.17 mm to (40.0, 12.7)
- moved R7 2.54 mm to (27.9, 5.08)
- moved C5 1.91 mm to (32.4, 7.62)
- moved C6 1.91 mm to (35.6, 7.62)
- moved JP8 0.32 mm to (59.1, 46.7)
Connections:
- net +12V: now also JP10.1, JP11.1, JP12.1, JP9.1
- net GND: now also JP10.2, JP11.2, JP12.2, JP9.2
- net RX: now also J1.RX, U$1.1; no longer U$1.2
- net TX: now also J1.TX, U$1.2; no longer U$1.1
Routing:
- net RX: track 0.00 -> 44.7 mm
- net TX: track 0.00 -> 41.1 mm
- net +12V: track 59.6 -> 86.0 mm
- net +5V: track 78.3 -> 55.8 mm
- net 5VA: track 41.7 -> 33.4 mm
- net AREF: track 47.2 -> 50.4 mm
- net AUDIO: track 7.40 -> 5.50 mm
- net A3: track 25.2 -> 23.3 mm
- net D13: track 20.2 -> 19.0 mm
- net N$999: track 5.72 -> 6.35 mm
- net N$6: track 3.81 -> 4.45 mm
Other:
- board text added: "v 2.0"
