File: Beta/eagle/tracker03-11.brd (EAGLE design)
At the start: 64.4 x 49.5 mm, 33 parts, among them IC1 7805, J1 ARRDUINO I, J2 7V-12V

Commit message: update
Parts:
- moved D1 1.42 mm to (10.8, 21.0)
- moved JP10 0.64 mm to (4.45, 21.6)
- moved JP11 0.64 mm to (4.45, 17.8)
- moved JP12 0.64 mm to (4.45, 29.2)
- moved J2 0.63 mm to (6.99, 10.8)
- moved JP9 0.63 mm to (4.45, 25.4)
- moved R6 0.63 mm to (21.0, 40.6)
Routing:
- net +12V: track 86.0 -> 84.6 mm
- net +5V: track 55.8 -> 54.6 mm
