File: eagle/tracker03-12.brd (EAGLE design)
At the start: 64.4 x 49.5 mm, 33 parts, among them IC1 7805, J1 ARRDUINO I, J2 7V-12V

Commit message: update
Parts:
- added JP13: (no value), pinhead:1X02
- ARDUINOII: value ARDUINO II -> ARDUINO_PRO_MINI
- moved C1 5.13 mm to (2.86, 40.6), turned to 270 degrees
- moved C2 4.51 mm to (8.57, 39.7)
- moved JP12 1.59 mm to (4.45, 27.6)
- moved JP9 1.27 mm to (4.45, 24.1)
- moved JP10 0.95 mm to (4.45, 20.6)
- moved JP11 0.64 mm to (4.45, 17.1)
- moved C4 0.32 mm to (14.3, 44.5)
- renumbered U$1 to ARDUINOII
Connections:
- new net D11A1: J1.D11, JP7.2, R8.2
- net +12V: now also JP13.1
- net D12: now also JP8.2, R9.2; no longer JP7.2, R8.2
- net D13: no longer JP8.2, R9.2
- net GND: now also JP13.2
Routing:
- net D11A1: track 0.00 -> 22.9 mm
- net D13: track 19.0 -> 0.00 mm
- net D12: track 15.5 -> 24.8 mm
- net +12V: track 84.6 -> 89.6 mm
Other:
- board text added: "github.com/QuadMax"
- board text added: "v3.2"
- board text removed: "v 2.0"
