File: eagle/tracker03-12.sch (EAGLE design)
At the start: 33 parts, among them IC1 7805, J1 ARRDUINO I, J2 7V-12V

Commit message: update
Parts:
- added JP13: (no value), pinhead:PINHD-1X2
- ARDUINOII: value ARDUINO II -> ARDUINO_PRO_MINI
- renumbered U$1 to ARDUINOII
Connections:
- new net D11A1: J1.*D11, JP7.2, R8.2
- net +12V: now also JP13.1
- net D12: now also JP8.2, R9.2; no longer JP7.2, R8.2
- net D13: no longer JP8.2, R9.2
- net GND: now also JP13.2
Changed lines of the file:
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@@
 <parts>
 <part name="J1" library="SparkFun-Boards" deviceset="ARDUINO_R3_SHIELD" device="NOLABELS" value="ARRDUINO I"/>
-<part name="U$1" library="SparkFun-Boards" deviceset="ARDUINO_PRO_MINI" device="" value="ARDUINO II"/>
+<part name="ARDUINOII" library="SparkFun-Boards" deviceset="ARDUINO_PRO_MINI" device="" value="ARDUINO_PRO_MINI"/>
 <part name="IC1" library="linear" deviceset="78*" device="TV" technology="05" value="7805"/>
 <part name="J2" library="con-jack" deviceset="JACK-PLUG" device="0" value="7V-12V"/>
@@
 <part name="P+16" library="supply1" deviceset="+12V" device=""/>
 <part name="GND17" library="supply1" deviceset="GND" device=""/>
+<part name="JP13" library="pinhead" deviceset="PINHD-1X2" device=""/>
+<part name="P+17" library="supply1" deviceset="+12V" device=""/>
+<part name="GND18" library="supply1" deviceset="GND" device=""/>
 </parts>
 <sheets>
@@
 <instances>
 <instance part="J1" gate="G$1" x="50.8" y="33.02"/>
-<instance part="U$1" gate="G$1" x="116.84" y="35.56"/>
+<instance part="ARDUINOII" gate="G$1" x="116.84" y="35.56"/>
 <instance part="IC1" gate="A1" x="2.54" y="55.88"/>
 <instance part="J2" gate="G$1" x="-30.48" y="53.34"/>
@@
 <instance part="P+16" gate="1" x="22.86" y="30.48" rot="R90"/>
 <instance part="GND17" gate="1" x="22.86" y="27.94" rot="R270"/>
+<instance part="JP13" gate="G$1" x="17.78" y="-7.62"/>
+<instance part="P+17" gate="1" x="12.7" y="-5.08" rot="R90"/>
+<instance part="GND18" gate="1" x="12.7" y="-7.62" rot="R270"/>
 </instances>
 <busses>
@@
 </segment>
 <segment>
-<pinref part="U$1" gate="G$1" pin="GND@2"/>
+<pinref part="ARDUINOII" gate="G$1" pin="GND@2"/>
 <wire x1="129.54" y1="48.26" x2="132.08" y2="48.26" width="0.1524" layer="91"/>
 </segment>
 <segment>
-<pinref part="U$1" gate="G$1" pin="GND"/>
+<pinref part="ARDUINOII" gate="G$1" pin="GND"/>
 <wire x1="106.68" y1="43.18" x2="104.14" y2="43.18" width="0.1524" layer="91"/>
 </segment>
@@
 <pinref part="JP12" gate="G$1" pin="2"/>
 <pinref part="GND17" gate="1" pin="GND"/>
+</segment>
+<segment>
+<pinref part="JP13" gate="G$1" pin="2"/>
+<pinref part="GND18" gate="1" pin="GND"/>
 </segment>
 </net>
@@
 </segment>
 <segment>
-<pinref part="U$1" gate="G$1" pin="2"/>
+<pinref part="ARDUINOII" gate="G$1" pin="2"/>
 <wire x1="106.68" y1="40.64" x2="104.14" y2="40.64" width="0.1524" layer="91"/>
 </segment>
@@
 <net name="D3" class="0">
 <segment>
-<pinref part="U$1" gate="G$1" pin="*3"/>
+<pinref part="ARDUINOII" gate="G$1" pin="*3"/>
 <wire x1="106.68" y1="38.1" x2="104.14" y2="38.1" width="0.1524" layer="91"/>
 </segment>
@@
 </segment>
 <segment>
-<pinref part="U$1" gate="G$1" pin="RAW"/>
+<pinref part="ARDUINOII" gate="G$1" pin="RAW"/>
 <pinref part="P+5" gate="1" pin="+12V"/>
 </segment>
@@
 <pinref part="P+16" gate="1" pin="+12V"/>
 </segment>
+<segment>
+<pinref part="JP13" gate="G$1" pin="1"/>
+<pinref part="P+17" gate="1" pin="+12V"/>
+</segment>
 </net>
 <net name="A4" class="0">
 <segment>
-<pinref part="U$1" gate="G$1" pin="A4"/>
+<pinref part="ARDUINOII" gate="G$1" pin="A4"/>
 <wire x1="106.68" y1="17.78" x2="104.14" y2="17.78" width="0.1524" layer="91"/>
 </segment>
@@
 <net name="A5" class="0">
 <segment>
-<pinref part="U$1" gate="G$1" pin="A5"/>
+<pinref part="ARDUINOII" gate="G$1" pin="A5"/>
 <wire x1="106.68" y1="15.24" x2="104.14" y2="15.24" width="0.1524" layer="91"/>
 </segment>
@@
 <net name="A2" class="0">
 <segment>
-<pinref part="U$1" gate="G$1" pin="A2"/>
+<pinref part="ARDUINOII" gate="G$1" pin="A2"/>
 <wire x1="129.54" y1="38.1" x2="132.08" y2="38.1" width="0.1524" layer="91"/>
 </segment>
@@
 </segment>
 <segment>
-<pinref part="U$1" gate="G$1" pin="TXO"/>
+<pinref part="ARDUINOII" gate="G$1" pin="TXO"/>
 <wire x1="106.68" y1="50.8" x2="104.14" y2="50.8" width="0.1524" layer="91"/>
 </segment>
@@
 </segment>
 <segment>
-<pinref part="U$1" gate="G$1" pin="RXI"/>
+<pinref part="ARDUINOII" gate="G$1" pin="RXI"/>
 <wire x1="106.68" y1="48.26" x2="104.14" y2="48.26" width="0.1524" layer="91"/>
 </segment>
@@
 <net name="D4" class="0">
 <segment>
-<pinref part="U$1" gate="G$1" pin="4"/>
+<pinref part="ARDUINOII" gate="G$1" pin="4"/>
 <wire x1="106.68" y1="35.56" x2="104.14" y2="35.56" width="0.1524" layer="91"/>
 </segment>
@@
 <net name="D11" class="0">
 <segment>
-<pinref part="U$1" gate="G$1" pin="*11"/>
+<pinref part="ARDUINOII" gate="G$1" pin="*11"/>
 <wire x1="129.54" y1="25.4" x2="132.08" y2="25.4" width="0.1524" layer="91"/>
 </segment>
@@
 <pinref part="J1" gate="G$1" pin="D12"/>
 <wire x1="63.5" y1="17.78" x2="66.04" y2="17.78" width="0.1524" layer="91"/>
+</segment>
+<segment>
+<pinref part="R9" gate="G$1" pin="2"/>
+<pinref part="JP8" gate="G$1" pin="2"/>
+<wire x1="78.74" y1="55.88" x2="83.82" y2="55.88" width="0.1524" layer="91"/>
+<wire x1="78.74" y1="55.88" x2="78.74" y2="53.34" width="0.1524" layer="91"/>
+</segment>
+</net>
+<net name="D13" class="0">
+<segment>
+<pinref part="J1" gate="G$1" pin="D13"/>
+<wire x1="63.5" y1="15.24" x2="66.04" y2="15.24" width="0.1524" layer="91"/>
+</segment>
+</net>
+<net name="D11A1" class="0">
+<segment>
+<pinref part="J1" gate="G$1" pin="*D11"/>
+<wire x1="63.5" y1="20.32" x2="66.04" y2="20.32" width="0.1524" layer="91"/>
 </segment>
 <segment>
@@
 </segment>
 </net>
-<net name="D13" class="0">
-<segment>
-<pinref part="J1" gate="G$1" pin="D13"/>
-<wire x1="63.5" y1="15.24" x2="66.04" y2="15.24" width="0.1524" layer="91"/>
-</segment>
-<segment>
-<pinref part="R9" gate="G$1" pin="2"/>
-<pinref part="JP8" gate="G$1" pin="2"/>
-<wire x1="78.74" y1="55.88" x2="83.82" y2="55.88" width="0.1524" layer="91"/>
-<wire x1="78.74" y1="55.88" x2="78.74" y2="53.34" width="0.1524" layer="91"/>
-</segment>
-</net>
